Commit message: 1869 urdf finished and roller mount attached

File: hiwin_ra610_1869_gb_support/urdf/ra610_1869-dexterity_gb_macro.xacro (robot description, xacro)
@@ -5,5 +5,5 @@
     <link name="${prefix}base_link" >
         <visual>
-            <origin xyz="0 0 0" rpy="0 0 ${pi/2}"/>
+            <origin xyz="0 0 0" rpy="0 0 0"/>
             <geometry>
                 <mesh filename="package://hiwin_ra610_1869_gb_support/meshes/RA610-1869-001.stl" scale="0.001 0.001 0.001"/>
@@ -14,5 +14,5 @@
         </visual>
         <collision>
-            <origin xyz="0 0 0" rpy="0 0 ${pi/2}"/>
+            <origin xyz="0 0 0" rpy="0 0 0"/>
             <geometry>
                 <mesh filename="package://hiwin_ra610_1869_gb_support/meshes/RA610-1869-001.stl" scale="0.001 0.001 0.001"/>
@@ -22,5 +22,5 @@
     <link name="${prefix}link_1" >
         <visual>
-            <origin xyz="0 0 0" rpy="0 0 ${pi/2}"/>
+            <origin xyz="0 0 0" rpy="0 0 0"/>
             <geometry>
                 <mesh filename="package://hiwin_ra610_1869_gb_support/meshes/RA610-1869-002.stl" scale="0.001 0.001 0.001"/>
@@ -31,13 +31,15 @@
         </visual>
         <collision>
-            <origin xyz="0 0 0" rpy="0 0 ${pi/2}"/>
+            <origin xyz="0 0 0" rpy="0 0 0"/>
             <geometry>
                 <mesh filename="package://hiwin_ra610_1869_gb_support/meshes/RA610-1869-002.stl" scale="0.001 0.001 0.001"/>
             </geometry>
+            <mass value="25.4709"/>
+            <inertia ixx="0.643616814" ixy="0.751558312" ixz="0.797091831" iyy="0.057618652" iyz="-0.180486233" izz="-0.019339033"/>
         </collision>
     </link>
     <link name="${prefix}link_2" >
         <visual>
-            <origin xyz="0 0 0" rpy="0 0 ${pi/2}"/>
+            <origin xyz="0 0 0" rpy="0 0 1.57"/>
             <geometry>
                 <mesh filename="package://hiwin_ra610_1869_gb_support/meshes/RA610-1869-003.stl" scale="0.001 0.001 0.001"/>
@@ -48,5 +50,5 @@
         </visual>
         <collision>
-            <origin xyz="0 0 0" rpy="0 0 ${pi/2}"/>
+            <origin xyz="0 0 0" rpy="0 0 1.57"/>
             <geometry>
                 <mesh filename="package://hiwin_ra610_1869_gb_support/meshes/RA610-1869-003.stl" scale="0.001 0.001 0.001"/>
@@ -56,5 +58,5 @@
     <link name="${prefix}link_3" >
         <visual>
-            <origin xyz="0 0 0" rpy="0 0 ${pi/2}"/>
+            <origin xyz="0 0 0" rpy="0 0 1.57"/>
             <geometry>
                 <mesh filename="package://hiwin_ra610_1869_gb_support/meshes/RA610-1869-004.stl" scale="0.001 0.001 0.001"/>
@@ -65,5 +67,5 @@
         </visual>
         <collision>
-            <origin xyz="0 0 0" rpy="0 0 ${pi/2}"/>
+            <origin xyz="0 0 0" rpy="0 0 1.57"/>
             <geometry>
                 <mesh filename="package://hiwin_ra610_1869_gb_support/meshes/RA610-1869-004.stl" scale="0.001 0.001 0.001"/>
@@ -73,5 +75,5 @@
     <link name="${prefix}link_4" >
         <visual>
-            <origin xyz="0 0 0" rpy="0 0 ${pi/2}"/>
+            <origin xyz="0 0 0" rpy="0 0 1.57"/>
             <geometry>
                 <mesh filename="package://hiwin_ra610_1869_gb_support/meshes/RA610-1869-005.stl" scale="0.001 0.001 0.001"/>
@@ -82,5 +84,5 @@
         </visual>
         <collision>
-            <origin xyz="0 0 0" rpy="0 0 ${pi/2}"/>
+            <origin xyz="0 0 0" rpy="0 0 1.57"/>
             <geometry>
                 <mesh filename="package://hiwin_ra610_1869_gb_support/meshes/RA610-1869-005.stl" scale="0.001 0.001 0.001"/>
@@ -90,5 +92,5 @@
     <link name="${prefix}link_5" >
         <visual>
-            <origin xyz="0 0 0" rpy="0 0 ${pi/2}"/>
+            <origin xyz="0 0 0" rpy="1.57 -1.57 1.57"/>
             <geometry>
                 <mesh filename="package://hiwin_ra610_1869_gb_support/meshes/RA610-1869-006.stl" scale="0.001 0.001 0.001"/>
@@ -99,5 +101,5 @@
         </visual>
         <collision>
-            <origin xyz="0 0 0" rpy="0 0 ${pi/2}"/>
+            <origin xyz="0 0 0" rpy="1.57 -1.57 1.57"/>
             <geometry>
                 <mesh filename="package://hiwin_ra610_1869_gb_support/meshes/RA610-1869-006.stl" scale="0.001 0.001 0.001"/>
@@ -107,5 +109,5 @@
     <link name="${prefix}link_6" >
         <visual>
-            <origin xyz="0 0 0" rpy="0 0 ${pi/2}"/>
+            <origin xyz="0 0 0" rpy="0 0 0"/>
             <geometry>
                 <mesh filename="package://hiwin_ra610_1869_gb_support/meshes/RA610-1869-007.stl" scale="0.001 0.001 0.001"/>
@@ -116,5 +118,5 @@
         </visual>
         <collision>
-            <origin xyz="0 0 0" rpy="0 0 ${pi/2}"/>
+            <origin xyz="0 0 0" rpy="0 0 0"/>
             <geometry>
                 <mesh filename="package://hiwin_ra610_1869_gb_support/meshes/RA610-1869-007.stl" scale="0.001 0.001 0.001"/>
@@ -122,46 +124,45 @@
         </collision>
     </link>
-    <!-- joints: main serial chain -->
     <joint name="${prefix}joint_1" type="revolute">
-        <origin xyz="0.0 0.0 0.191" rpy="0.0 0.0 0.0" />
+        <origin xyz="0.0 0.0 0.1965" rpy="0.0 0.0 0.0" />
         <parent link="${prefix}base_link" />
         <child link="${prefix}link_1" />
         <axis xyz="0 0 1" />
-        <limit lower="-2.8792" upper="2.8792" effort="0" velocity="2.618"/>
+        <limit lower="-2.967" upper="2.967" effort="0" velocity="2.618"/>
     </joint>
     <joint name="${prefix}joint_2" type="revolute">
-        <origin xyz="0.0 0.140 0.255" rpy="0.0 0.0 0.0" />
+        <origin xyz="0.140 -0.099 0.252" rpy="1.57 0 0" />
         <parent link="${prefix}link_1" />
         <child link="${prefix}link_2" />
-        <axis xyz="1 0 0" />
+        <axis xyz="0 0 1" />
         <limit lower="-2.1812" upper="1.4832" effort="0" velocity="2.618"/>
     </joint>
     <joint name="${prefix}joint_3" type="revolute">
-        <origin xyz="0.0 0.000 0.642" rpy="0.0 0.0 0.0" />
+        <origin xyz="0 0.640 -0.094" rpy="0.0 0.0 0.0" />
         <parent link="${prefix}link_2" />
         <child link="${prefix}link_3" />
-        <axis xyz="1 0 0" />
-        <limit lower="-0.9597" upper="3.2282" effort="0" velocity="2.618"/>
+        <axis xyz="0 0 1" />
+        <limit lower="-1.483" upper="3.228" effort="0" velocity="3.829"/>
     </joint>
     <joint name="${prefix}joint_4" type="revolute">
-        <origin xyz="0.0 0.1495 0.160" rpy="0.0 0.0 0.0" />
+        <origin xyz="0.231 0.160 0.005" rpy="0 1.57 0.0" />
         <parent link="${prefix}link_3" />
         <child link="${prefix}link_4" />
-        <axis xyz="0 1 0" />
-        <limit lower="-3.3155" upper="3.3155" effort="0" velocity="2.618"/>
+        <axis xyz="0 0 1" />
+        <limit lower="-3.3155" upper="3.3155" effort="0" velocity="7.757"/>
     </joint>
     <joint name="${prefix}joint_5" type="revolute">
-        <origin xyz="0.0 0.4025 0.000" rpy="0.0 0.0 0.0" />
+        <origin xyz="0 0 0.847" rpy="0 0.0 0" />
         <parent link="${prefix}link_4" />
         <child link="${prefix}link_5" />
-        <axis xyz="1 0 0" />
-        <limit lower="-2.0067" upper="2.0067" effort="0" velocity="2.618"/>
+        <axis xyz="0 0 1" />
+        <limit lower="-2.356" upper="2.356" effort="0" velocity="7.853"/>
     </joint>
     <joint name="${prefix}joint_6" type="revolute">
-        <origin xyz="0.0 0.080 0.0" rpy="0.0 0.0 0.0" />
+        <origin xyz="0.0 0.0 0.101" rpy="0 0 0" />
         <parent link="${prefix}link_5" />
         <child link="${prefix}link_6" />
-        <axis xyz="0 1 0" />
-        <limit lower="-3.1415" upper="3.1415" effort="0" velocity="2.618"/>
+        <axis xyz="0 0 1" />
+        <limit lower="-6.28" upper="6.28" effort="0" velocity="12.566"/>
     </joint>
     <!-- ROS-Industrial 'base' frame: base_link to HIWIN World Coordinates transform -->
@@ -175,5 +176,5 @@
     <link name="${prefix}flange" />
     <joint name="${prefix}joint_6-flange" type="fixed">
-      <origin xyz="0 0.016 0" rpy="0 0 0" />
+      <origin xyz="0 0. 0.016" rpy="0 0 0" />
       <parent link="${prefix}link_6" />
       <child link="${prefix}flange" />
@@ -182,5 +183,5 @@
     <link name="${prefix}tool0" />
     <joint name="${prefix}link_6-tool0" type="fixed">
-      <origin xyz="0 0.020 0.0" rpy="0.0 ${-pi/2.0} ${-pi/2.0}" />
+      <origin xyz="0 0 0.020" rpy="0.0 ${-pi/2.0} ${-pi/2.0}" />
       <parent link="${prefix}link_6" />
       <child link="${prefix}tool0" />

File: hiwin_ra610_1869_gb_support/urdf/ra610_1869_gb.xacro (robot description, xacro)
@@ -1,5 +1,5 @@
 <?xml version="1.0"?>
 <robot xmlns:xacro="http://ros.org/wiki/xacro" name="manipulator" >
-  <xacro:include filename="$(find hiwin_ra610_1869_gb_support)/urdf/ra610_1869_gb_macro2.xacro" />
+  <xacro:include filename="$(find hiwin_ra610_1869_gb_support)/urdf/ra610_1869_gb_macro.xacro" />
   <xacro:manipulator prefix="" />
 </robot>

File: hiwin_ra610_1869_gb_support/urdf/ra610_1869_gb_macro.xacro (robot description, xacro)
@@ -5,5 +5,5 @@
     <link name="${prefix}base_link" >
         <visual>
-            <origin xyz="0 0 0" rpy="0 0 0"/>
+            <origin xyz="0 0 0" rpy="0 0 ${pi/2}"/>
             <geometry>
                 <mesh filename="package://hiwin_ra610_1869_gb_support/meshes/RA610-1869-001.stl" scale="0.001 0.001 0.001"/>
@@ -14,5 +14,5 @@
         </visual>
         <collision>
-            <origin xyz="0 0 0" rpy="0 0 0"/>
+            <origin xyz="0 0 0" rpy="0 0 ${pi/2}"/>
             <geometry>
                 <mesh filename="package://hiwin_ra610_1869_gb_support/meshes/RA610-1869-001.stl" scale="0.001 0.001 0.001"/>
@@ -22,5 +22,5 @@
     <link name="${prefix}link_1" >
         <visual>
-            <origin xyz="0 0 0" rpy="0 0 0"/>
+            <origin xyz="0 0 0" rpy="0 0 ${pi/2}"/>
             <geometry>
                 <mesh filename="package://hiwin_ra610_1869_gb_support/meshes/RA610-1869-002.stl" scale="0.001 0.001 0.001"/>
@@ -31,15 +31,13 @@
         </visual>
         <collision>
-            <origin xyz="0 0 0" rpy="0 0 0"/>
+            <origin xyz="0 0 0" rpy="0 0 ${pi/2}"/>
             <geometry>
                 <mesh filename="package://hiwin_ra610_1869_gb_support/meshes/RA610-1869-002.stl" scale="0.001 0.001 0.001"/>
             </geometry>
-            <mass value="25.4709"/>
-            <inertia ixx="0.643616814" ixy="0.751558312" ixz="0.797091831" iyy="0.057618652" iyz="-0.180486233" izz="-0.019339033"/>
         </collision>
     </link>
     <link name="${prefix}link_2" >
         <visual>
-            <origin xyz="0 0 0" rpy="0 0 1.57"/>
+            <origin xyz="0 0 0" rpy="${pi} ${-pi/2} 0"/>
             <geometry>
                 <mesh filename="package://hiwin_ra610_1869_gb_support/meshes/RA610-1869-003.stl" scale="0.001 0.001 0.001"/>
@@ -50,5 +48,5 @@
         </visual>
         <collision>
-            <origin xyz="0 0 0" rpy="0 0 1.57"/>
+            <origin xyz="0 0 0" rpy="${pi} ${-pi/2} 0"/>
             <geometry>
                 <mesh filename="package://hiwin_ra610_1869_gb_support/meshes/RA610-1869-003.stl" scale="0.001 0.001 0.001"/>
@@ -58,5 +56,5 @@
     <link name="${prefix}link_3" >
         <visual>
-            <origin xyz="0 0 0" rpy="0 0 1.57"/>
+            <origin xyz="0 0 0" rpy="${pi} ${-pi/2} 0"/>
             <geometry>
                 <mesh filename="package://hiwin_ra610_1869_gb_support/meshes/RA610-1869-004.stl" scale="0.001 0.001 0.001"/>
@@ -67,5 +65,5 @@
         </visual>
         <collision>
-            <origin xyz="0 0 0" rpy="0 0 1.57"/>
+            <origin xyz="0 0 0" rpy="${pi} ${-pi/2} 0"/>
             <geometry>
                 <mesh filename="package://hiwin_ra610_1869_gb_support/meshes/RA610-1869-004.stl" scale="0.001 0.001 0.001"/>
@@ -75,5 +73,5 @@
     <link name="${prefix}link_4" >
         <visual>
-            <origin xyz="0 0 0" rpy="0 0 1.57"/>
+            <origin xyz="0 0 0" rpy="0 ${-pi/2} ${-pi/2}"/>
             <geometry>
                 <mesh filename="package://hiwin_ra610_1869_gb_support/meshes/RA610-1869-005.stl" scale="0.001 0.001 0.001"/>
@@ -84,5 +82,5 @@
         </visual>
         <collision>
-            <origin xyz="0 0 0" rpy="0 0 1.57"/>
+            <origin xyz="0 0 0" rpy="0 ${-pi/2} ${-pi/2}"/>
             <geometry>
                 <mesh filename="package://hiwin_ra610_1869_gb_support/meshes/RA610-1869-005.stl" scale="0.001 0.001 0.001"/>
@@ -92,5 +90,5 @@
     <link name="${prefix}link_5" >
         <visual>
-            <origin xyz="0 0 0" rpy="1.57 -1.57 1.57"/>
+            <origin xyz="0 0 0" rpy="${pi/2} 0 ${pi/2}"/>
             <geometry>
                 <mesh filename="package://hiwin_ra610_1869_gb_support/meshes/RA610-1869-006.stl" scale="0.001 0.001 0.001"/>
@@ -101,5 +99,5 @@
         </visual>
         <collision>
-            <origin xyz="0 0 0" rpy="1.57 -1.57 1.57"/>
+            <origin xyz="0 0 0" rpy="${pi/2} 0 ${pi/2}"/>
             <geometry>
                 <mesh filename="package://hiwin_ra610_1869_gb_support/meshes/RA610-1869-006.stl" scale="0.001 0.001 0.001"/>
@@ -109,5 +107,5 @@
     <link name="${prefix}link_6" >
         <visual>
-            <origin xyz="0 0 0" rpy="0 0 0"/>
+            <origin xyz="0 0 0" rpy="0 ${-pi/2} ${-pi/2}"/>
             <geometry>
                 <mesh filename="package://hiwin_ra610_1869_gb_support/meshes/RA610-1869-007.stl" scale="0.001 0.001 0.001"/>
@@ -118,5 +116,5 @@
         </visual>
         <collision>
-            <origin xyz="0 0 0" rpy="0 0 0"/>
+            <origin xyz="0 0 0" rpy="0 0 ${pi/2}"/>
             <geometry>
                 <mesh filename="package://hiwin_ra610_1869_gb_support/meshes/RA610-1869-007.stl" scale="0.001 0.001 0.001"/>
@@ -124,4 +122,5 @@
         </collision>
     </link>
+    <!-- joints: main serial chain -->
     <joint name="${prefix}joint_1" type="revolute">
         <origin xyz="0.0 0.0 0.1965" rpy="0.0 0.0 0.0" />
@@ -132,36 +131,36 @@
     </joint>
     <joint name="${prefix}joint_2" type="revolute">
-        <origin xyz="0.140 -0.099 0.252" rpy="1.57 0 0" />
+        <origin xyz="0.094 0.140 0.252" rpy="0.0 0.0 0.0" />
         <parent link="${prefix}link_1" />
         <child link="${prefix}link_2" />
-        <axis xyz="0 0 1" />
+        <axis xyz="1 0 0" />
         <limit lower="-2.1812" upper="1.4832" effort="0" velocity="2.618"/>
     </joint>
     <joint name="${prefix}joint_3" type="revolute">
-        <origin xyz="0 0.640 -0.094" rpy="0.0 0.0 0.0" />
+        <origin xyz="-0.094 0 0.640" rpy="0.0 0.0 0.0" />
         <parent link="${prefix}link_2" />
         <child link="${prefix}link_3" />
-        <axis xyz="0 0 1" />
+        <axis xyz="1 0 0" />
         <limit lower="-1.483" upper="3.228" effort="0" velocity="3.829"/>
     </joint>
     <joint name="${prefix}joint_4" type="revolute">
-        <origin xyz="0.231 0.160 0.005" rpy="0 1.57 0.0" />
+        <origin xyz="-0.005 0.231 0.160" rpy="0.0 0.0 0.0" />
         <parent link="${prefix}link_3" />
         <child link="${prefix}link_4" />
-        <axis xyz="0 0 1" />
+        <axis xyz="0 1 0" />
         <limit lower="-3.3155" upper="3.3155" effort="0" velocity="7.757"/>
     </joint>
     <joint name="${prefix}joint_5" type="revolute">
-        <origin xyz="0 0 0.847" rpy="0 0.0 0" />
+        <origin xyz="0.0 0.847 0.000" rpy="0.0 0.0 0.0" />
         <parent link="${prefix}link_4" />
         <child link="${prefix}link_5" />
-        <axis xyz="0 0 1" />
+        <axis xyz="1 0 0" />
         <limit lower="-2.356" upper="2.356" effort="0" velocity="7.853"/>
     </joint>
     <joint name="${prefix}joint_6" type="revolute">
-        <origin xyz="0.0 0.0 0.101" rpy="0 0 0" />
+        <origin xyz="0.0 0.101 0.0" rpy="0.0 0.0 0.0" />
         <parent link="${prefix}link_5" />
         <child link="${prefix}link_6" />
-        <axis xyz="0 0 1" />
+        <axis xyz="0 1 0" />
         <limit lower="-6.28" upper="6.28" effort="0" velocity="12.566"/>
     </joint>
@@ -176,5 +175,5 @@
     <link name="${prefix}flange" />
     <joint name="${prefix}joint_6-flange" type="fixed">
-      <origin xyz="0 0. 0.016" rpy="0 0 0" />
+      <origin xyz="0 0.016 0" rpy="0 0 0" />
       <parent link="${prefix}link_6" />
       <child link="${prefix}flange" />
@@ -183,5 +182,6 @@
     <link name="${prefix}tool0" />
     <joint name="${prefix}link_6-tool0" type="fixed">
-      <origin xyz="0 0 0.020" rpy="0.0 ${-pi/2.0} ${-pi/2.0}" />
+      <!-- <origin xyz="0 0.020 0.0" rpy="0.0 ${-pi/2.0} ${-pi/2.0}" /> -->
+        <origin xyz="0 0.020 0.0" rpy="0.0 0.0 0.0" />
       <parent link="${prefix}link_6" />
       <child link="${prefix}tool0" />
