Commit message: my urdf implemented

File: hiwin_ra610_1869_gb_support/urdf/ra610_1869_gb_macro.xacro (robot description, xacro)
@@ -5,5 +5,5 @@
     <link name="${prefix}base_link" >
         <visual>
-            <origin xyz="0 0 0" rpy="0 0 ${pi/2}"/>
+            <origin xyz="0 0 0" rpy="0 0 0"/>
             <geometry>
                 <mesh filename="package://hiwin_ra610_1869_gb_support/meshes/RA610-1869-001.obj" scale="0.001 0.001 0.001"/>
@@ -14,5 +14,5 @@
         </visual>
         <collision>
-            <origin xyz="0 0 0" rpy="0 0 ${pi/2}"/>
+            <origin xyz="0 0 0" rpy="0 0 0"/>
             <geometry>
                 <mesh filename="package://hiwin_ra610_1869_gb_support/meshes/RA610-1869-001.obj" scale="0.001 0.001 0.001"/>
@@ -22,5 +22,5 @@
     <link name="${prefix}link_1" >
         <visual>
-            <origin xyz="0 0 0" rpy="0 0 ${pi/2}"/>
+            <origin xyz="0 0 0" rpy="0 0 0"/>
             <geometry>
                 <mesh filename="package://hiwin_ra610_1869_gb_support/meshes/RA610-1869-002.obj" scale="0.001 0.001 0.001"/>
@@ -31,15 +31,17 @@
         </visual>
         <collision>
-            <origin xyz="0 0 0" rpy="0 0 ${pi/2}"/>
+            <origin xyz="0 0 0" rpy="0 0 0"/>
             <geometry>
-                <mesh filename="package://hiwin_ra610_1869_gb_support/meshes/RA610-1869-001.obj" scale="0.001 0.001 0.001"/>
+                <mesh filename="package://hiwin_ra610_1869_gb_support/meshes/RA610-1869-002.obj" scale="0.001 0.001 0.001"/>
             </geometry>
+            <mass value="25.4709"/>
+            <inertia ixx="0.643616814" ixy="0.751558312" ixz="0.797091831" iyy="0.057618652" iyz="-0.180486233" izz="-0.019339033"/>
         </collision>
     </link>
     <link name="${prefix}link_2" >
         <visual>
-            <origin xyz="0 0 0" rpy="0 0 ${pi/2}"/>
+            <origin xyz="0 0 0" rpy="0 0 1.57"/>
             <geometry>
-                <mesh filename="package://hiwin_ra610_1355_gb_support/meshes/visual/link_2.stl" scale="0.001 0.001 0.001"/>
+                <mesh filename="package://hiwin_ra610_1869_gb_support/meshes/RA610-1869-003.obj" scale="0.001 0.001 0.001"/>
             </geometry>
             <material name="LightGrey">
@@ -48,7 +50,7 @@
         </visual>
         <collision>
-            <origin xyz="0 0 0" rpy="0 0 ${pi/2}"/>
+            <origin xyz="0 0 0" rpy="0 0 1.57"/>
             <geometry>
-                <mesh filename="package://hiwin_ra610_1355_gb_support/meshes/collision/link_2.stl" scale="0.001 0.001 0.001"/>
+                <mesh filename="package://hiwin_ra610_1869_gb_support/meshes/RA610-1869-003.obj" scale="0.001 0.001 0.001"/>
             </geometry>
         </collision>
@@ -56,7 +58,7 @@
     <link name="${prefix}link_3" >
         <visual>
-            <origin xyz="0 0 0" rpy="0 0 ${pi/2}"/>
+            <origin xyz="0 0 0" rpy="0 0 1.57"/>
             <geometry>
-                <mesh filename="package://hiwin_ra610_1355_gb_support/meshes/visual/link_3.stl" scale="0.001 0.001 0.001"/>
+                <mesh filename="package://hiwin_ra610_1869_gb_support/meshes/RA610-1869-004.obj" scale="0.001 0.001 0.001"/>
             </geometry>
             <material name="LightGrey">
@@ -65,7 +67,7 @@
         </visual>
         <collision>
-            <origin xyz="0 0 0" rpy="0 0 ${pi/2}"/>
+            <origin xyz="0 0 0" rpy="0 0 1.57"/>
             <geometry>
-                <mesh filename="package://hiwin_ra610_1355_gb_support/meshes/collision/link_3.stl" scale="0.001 0.001 0.001"/>
+                <mesh filename="package://hiwin_ra610_1869_gb_support/meshes/RA610-1869-004.obj" scale="0.001 0.001 0.001"/>
             </geometry>
         </collision>
@@ -73,7 +75,7 @@
     <link name="${prefix}link_4" >
         <visual>
-            <origin xyz="0 0 0" rpy="0 0 ${pi/2}"/>
+            <origin xyz="0 0 0" rpy="0 0 1.57"/>
             <geometry>
-                <mesh filename="package://hiwin_ra610_1355_gb_support/meshes/visual/link_4.stl" scale="0.001 0.001 0.001"/>
+                <mesh filename="package://hiwin_ra610_1869_gb_support/meshes/RA610-1869-005.obj" scale="0.001 0.001 0.001"/>
             </geometry>
             <material name="LightGrey">
@@ -82,7 +84,7 @@
         </visual>
         <collision>
-            <origin xyz="0 0 0" rpy="0 0 ${pi/2}"/>
+            <origin xyz="0 0 0" rpy="0 0 1.57"/>
             <geometry>
-                <mesh filename="package://hiwin_ra610_1355_gb_support/meshes/collision/link_4.stl" scale="0.001 0.001 0.001"/>
+                <mesh filename="package://hiwin_ra610_1869_gb_support/meshes/RA610-1869-005.obj" scale="0.001 0.001 0.001"/>
             </geometry>
         </collision>
@@ -90,7 +92,7 @@
     <link name="${prefix}link_5" >
         <visual>
-            <origin xyz="0 0 0" rpy="0 0 ${pi/2}"/>
+            <origin xyz="0 0 0" rpy="1.57 -1.57 1.57"/>
             <geometry>
-                <mesh filename="package://hiwin_ra610_1355_gb_support/meshes/visual/link_5.stl" scale="0.001 0.001 0.001"/>
+                <mesh filename="package://hiwin_ra610_1869_gb_support/meshes/RA610-1869-006.obj" scale="0.001 0.001 0.001"/>
             </geometry>
             <material name="LightGrey">
@@ -99,7 +101,7 @@
         </visual>
         <collision>
-            <origin xyz="0 0 0" rpy="0 0 ${pi/2}"/>
+            <origin xyz="0 0 0" rpy="1.57 -1.57 1.57"/>
             <geometry>
-                <mesh filename="package://hiwin_ra610_1355_gb_support/meshes/collision/link_5.stl" scale="0.001 0.001 0.001"/>
+                <mesh filename="package://hiwin_ra610_1869_gb_support/meshes/RA610-1869-006.obj" scale="0.001 0.001 0.001"/>
             </geometry>
         </collision>
@@ -107,7 +109,7 @@
     <link name="${prefix}link_6" >
         <visual>
-            <origin xyz="0 0 0" rpy="0 0 ${pi/2}"/>
+            <origin xyz="0 0 0" rpy="0 0 0"/>
             <geometry>
-                <mesh filename="package://hiwin_ra610_1355_gb_support/meshes/visual/link_6.stl" scale="0.001 0.001 0.001"/>
+                <mesh filename="package://hiwin_ra610_1869_gb_support/meshes/RA610-1869-007.obj" scale="0.001 0.001 0.001"/>
             </geometry>
             <material name="LightGrey">
@@ -116,11 +118,10 @@
         </visual>
         <collision>
-            <origin xyz="0 0 0" rpy="0 0 ${pi/2}"/>
+            <origin xyz="0 0 0" rpy="0 0 0"/>
             <geometry>
-                <mesh filename="package://hiwin_ra610_1355_gb_support/meshes/collision/link_6.stl" scale="0.001 0.001 0.001"/>
+                <mesh filename="package://hiwin_ra610_1869_gb_support/meshes/RA610-1869-007.obj" scale="0.001 0.001 0.001"/>
             </geometry>
         </collision>
     </link>
-    <!-- joints: main serial chain -->
     <joint name="${prefix}joint_1" type="revolute">
         <origin xyz="0.0 0.0 0.1965" rpy="0.0 0.0 0.0" />
@@ -128,40 +129,40 @@
         <child link="${prefix}link_1" />
         <axis xyz="0 0 1" />
-        <limit lower="-2.8792" upper="2.8792" effort="0" velocity="2.618"/>
+        <limit lower="-2.967" upper="2.967" effort="0" velocity="2.618"/>
     </joint>
     <joint name="${prefix}joint_2" type="revolute">
-        <origin xyz="0.0 0.140 0.255" rpy="0.0 0.0 0.0" />
+        <origin xyz="0.140 -0.099 0.252" rpy="1.57 0 0" />
         <parent link="${prefix}link_1" />
         <child link="${prefix}link_2" />
-        <axis xyz="1 0 0" />
+        <axis xyz="0 0 1" />
         <limit lower="-2.1812" upper="1.4832" effort="0" velocity="2.618"/>
     </joint>
     <joint name="${prefix}joint_3" type="revolute">
-        <origin xyz="0.0 0.000 0.642" rpy="0.0 0.0 0.0" />
+        <origin xyz="0 0.640 -0.094" rpy="0.0 0.0 0.0" />
         <parent link="${prefix}link_2" />
         <child link="${prefix}link_3" />
-        <axis xyz="1 0 0" />
-        <limit lower="-0.9597" upper="3.2282" effort="0" velocity="2.618"/>
+        <axis xyz="0 0 1" />
+        <limit lower="-1.483" upper="3.228" effort="0" velocity="3.829"/>
     </joint>
     <joint name="${prefix}joint_4" type="revolute">
-        <origin xyz="0.0 0.1495 0.160" rpy="0.0 0.0 0.0" />
+        <origin xyz="0.231 0.160 0.005" rpy="0 1.57 0.0" />
         <parent link="${prefix}link_3" />
         <child link="${prefix}link_4" />
-        <axis xyz="0 1 0" />
-        <limit lower="-3.3155" upper="3.3155" effort="0" velocity="2.618"/>
+        <axis xyz="0 0 1" />
+        <limit lower="-3.3155" upper="3.3155" effort="0" velocity="7.757"/>
     </joint>
     <joint name="${prefix}joint_5" type="revolute">
-        <origin xyz="0.0 0.4025 0.000" rpy="0.0 0.0 0.0" />
+        <origin xyz="0 0 0.847" rpy="0 0.0 0" />
         <parent link="${prefix}link_4" />
         <child link="${prefix}link_5" />
-        <axis xyz="1 0 0" />
-        <limit lower="-2.0067" upper="2.0067" effort="0" velocity="2.618"/>
+        <axis xyz="0 0 1" />
+        <limit lower="-2.356" upper="2.356" effort="0" velocity="7.853"/>
     </joint>
     <joint name="${prefix}joint_6" type="revolute">
-        <origin xyz="0.0 0.080 0.0" rpy="0.0 0.0 0.0" />
+        <origin xyz="0.0 0.0 0.101" rpy="0 0 0" />
         <parent link="${prefix}link_5" />
         <child link="${prefix}link_6" />
-        <axis xyz="0 1 0" />
-        <limit lower="-3.1415" upper="3.1415" effort="0" velocity="2.618"/>
+        <axis xyz="0 0 1" />
+        <limit lower="-6.28" upper="6.28" effort="0" velocity="12.566"/>
     </joint>
     <!-- ROS-Industrial 'base' frame: base_link to HIWIN World Coordinates transform -->
@@ -175,5 +176,5 @@
     <link name="${prefix}flange" />
     <joint name="${prefix}joint_6-flange" type="fixed">
-      <origin xyz="0 0.016 0" rpy="0 0 0" />
+      <origin xyz="0 0. 0.016" rpy="0 0 0" />
       <parent link="${prefix}link_6" />
       <child link="${prefix}flange" />
@@ -182,5 +183,5 @@
     <link name="${prefix}tool0" />
     <joint name="${prefix}link_6-tool0" type="fixed">
-      <origin xyz="0 0.020 0.0" rpy="0.0 ${-pi/2.0} ${-pi/2.0}" />
+      <origin xyz="0 0 0.020" rpy="0.0 ${-pi/2.0} ${-pi/2.0}" />
       <parent link="${prefix}link_6" />
       <child link="${prefix}tool0" />

Commit message: hand_gesture_recognition

File: hiwin_ra610_1869_gb_support/urdf/ra610_1869_gb_macro.xacro (robot description, xacro)
@@ -122,4 +122,6 @@
         </collision>
     </link>
+    <!-- end_effector frame -->
+    <link name="${prefix}end_effector" />
     <!-- joints: main serial chain -->
     <joint name="${prefix}joint_1" type="revolute">
@@ -165,4 +167,9 @@
         <limit lower="-6.28" upper="6.28" effort="0" velocity="12.566"/>
     </joint>
+    <joint name="${prefix}end_effector" type="fixed">
+        <origin xyz="0 0.480 0.0" rpy="0.0 0.0 0.0" />
+        <parent link="${prefix}link_6" />
+        <child link="${prefix}end_effector" />
+    </joint>
     <!-- ROS-Industrial 'base' frame: base_link to HIWIN World Coordinates transform -->
     <link name="${prefix}base" />
@@ -175,5 +182,5 @@
     <link name="${prefix}flange" />
     <joint name="${prefix}joint_6-flange" type="fixed">
-      <origin xyz="0 0.016 0" rpy="0 0 0" />
+      <origin xyz="0 0 0" rpy="0 0 0" />
       <parent link="${prefix}link_6" />
       <child link="${prefix}flange" />
@@ -183,5 +190,5 @@
     <joint name="${prefix}link_6-tool0" type="fixed">
       <!-- <origin xyz="0 0.020 0.0" rpy="0.0 ${-pi/2.0} ${-pi/2.0}" /> -->
-        <origin xyz="0 0.020 0.0" rpy="0.0 0.0 0.0" />
+        <origin xyz="0 0.480 0.0" rpy="0.0 0.0 0.0" />
       <parent link="${prefix}link_6" />
       <child link="${prefix}tool0" />

File: hiwin_roller_support/urdf/roller_macro.xacro (robot description, xacro)
@@ -5,7 +5,7 @@
     <link name="${prefix}base_link">
         <visual>
-            <origin xyz="0 0.00 0" rpy="${-pi/2} ${pi} 0"/>
+            <origin xyz="0 0 0" rpy="${pi/2} 0 ${pi}"/>
             <geometry>
-                <mesh filename="package://hiwin_roller_support/meshes/roller_mount.stl"/>
+                <mesh filename="package://hiwin_roller_support/meshes/roller_mount.stl"  />
             </geometry>
             <material name="LightGrey">
@@ -14,11 +14,26 @@
         </visual>
         <collision>
-            <origin xyz="0 0.00625 0" rpy="0 0 ${pi}"/>
+            <origin xyz="0 0 0" rpy="${pi/2} 0 ${pi}"/>
             <geometry>
-                <mesh filename="package://hiwin_roller_support/meshes/roller_mount.stl" scale="0.001 0.001 0.001"/>
+                <mesh filename="package://hiwin_roller_support/meshes/roller_mount.stl" />
             </geometry>
         </collision>
     </link>
     <link name="${prefix}link_1" >
+        <visual>
+            <origin xyz="0.0 0.0 0.0" rpy="${pi/2} ${pi} 0"/>
+            <geometry>
+                <mesh filename="package://hiwin_roller_support/meshes/roller.stl" scale="0.001 0.001 0.001"/>
+            </geometry>
+            <material name="LightGrey">
+                <color rgba="0.7 0.7 0.7 1.0"/>
+            </material>
+        </visual>
+        <collision>
+            <origin xyz="0.0 0.0 0.0" rpy="${pi/2} 0 0"/>
+            <geometry>
+                <mesh filename="package://hiwin_roller_support/meshes/roller.stl" scale="0.001 0.001 0.001"/>
+            </geometry>
+        </collision>
     </link>
     <link name="${prefix}finger_1" >
@@ -28,21 +43,21 @@
     <!-- joints: main serial chain -->
     <joint name="${prefix}joint_1" type="fixed">
-        <origin xyz="0.002 0.0325 0.0" rpy="${pi} 0.0 0.0" />
+        <origin xyz="0.0 0. 0.0" rpy="${pi} 0.0 0.0" />
         <parent link="${prefix}base_link" />
         <child link="${prefix}link_1" />
     </joint>
     <joint name="${prefix}joint_finger_1" type="prismatic">
-      <origin xyz="0 0 0" rpy="0 0 0" />
+      <origin xyz="0.0 0 0" rpy="0 0 0" />
       <parent link="${prefix}link_1" />
       <child link="${prefix}finger_1" />
       <axis xyz="-1 0 0"/>
-      <limit lower="0.0" upper="0.008" effort="0" velocity="0.01"/>
+      <limit lower="0.0" upper="0.016" effort="0" velocity="0.01"/>
     </joint>
     <joint name="${prefix}joint_finger_2" type="prismatic">
-      <origin xyz="0.018 0 0" rpy="0 0 0" />
+      <origin xyz="0 0 0" rpy="0 0 0" />
       <parent link="${prefix}link_1" />
       <child link="${prefix}finger_2" />
       <axis xyz="1 0 0"/>
-      <limit lower="0.0" upper="0.008" effort="0" velocity="0.01"/>
+      <limit lower="0.0" upper="0.016" effort="0" velocity="0.01"/>
     </joint>
   </xacro:macro>

Commit message: final demo implemented

File: hiwin_ra610_1869_gb_support/urdf/ra610_1869_gb_macro.xacro (robot description, xacro)
@@ -194,4 +194,12 @@
       <child link="${prefix}tool0" />
     </joint>
+        <!-- ROS-Industrial 'tool0' frame: all-zeros tool frame -->
+    <link name="${prefix}ee_link" />
+    <joint name="${prefix}ee_joint" type="fixed">
+      <!-- <origin xyz="0 0.020 0.0" rpy="0.0 ${-pi/2.0} ${-pi/2.0}" /> -->
+        <origin xyz="0 0.480 0.0" rpy="0.0 0.0 0.0" />
+      <parent link="${prefix}link_6" />
+      <child link="${prefix}ee_link" />
+    </joint>
   </xacro:macro>
 </robot>

Commit message: 3d model changes

File: hiwin_ra610_1869_gb_support/urdf/ra610_1869_gb_macro.xacro (robot description, xacro)
@@ -130,5 +130,5 @@
         <child link="${prefix}link_1" />
         <axis xyz="0 0 1" />
-        <limit lower="-2.967" upper="2.967" effort="0" velocity="2.618"/>
+        <limit lower="-2.967" upper="2.967" effort="0" velocity="3.35103"/>
     </joint>
     <joint name="${prefix}joint_2" type="revolute">
@@ -137,5 +137,5 @@
         <child link="${prefix}link_2" />
         <axis xyz="1 0 0" />
-        <limit lower="-2.1812" upper="1.4832" effort="0" velocity="2.618"/>
+        <limit lower="-2.1812" upper="1.4832" effort="0" velocity="3.59538"/>
     </joint>
     <joint name="${prefix}joint_3" type="revolute">
@@ -144,5 +144,5 @@
         <child link="${prefix}link_3" />
         <axis xyz="1 0 0" />
-        <limit lower="-1.483" upper="3.228" effort="0" velocity="3.829"/>
+        <limit lower="-1.483" upper="3.228" effort="0" velocity="3.822"/>
     </joint>
     <joint name="${prefix}joint_4" type="revolute">
@@ -151,5 +151,5 @@
         <child link="${prefix}link_4" />
         <axis xyz="0 1 0" />
-        <limit lower="-3.3155" upper="3.3155" effort="0" velocity="7.757"/>
+        <limit lower="-3.3155" upper="3.3155" effort="0" velocity="7.853"/>
     </joint>
     <joint name="${prefix}joint_5" type="revolute">
@@ -168,5 +168,5 @@
     </joint>
     <joint name="${prefix}end_effector" type="fixed">
-        <origin xyz="0 0.480 0.0" rpy="0.0 0.0 0.0" />
+        <origin xyz="0 0.450 0.0" rpy="0.0 0.0 0.0" />
         <parent link="${prefix}link_6" />
         <child link="${prefix}end_effector" />
@@ -190,16 +190,8 @@
     <joint name="${prefix}link_6-tool0" type="fixed">
       <!-- <origin xyz="0 0.020 0.0" rpy="0.0 ${-pi/2.0} ${-pi/2.0}" /> -->
-        <origin xyz="0 0.480 0.0" rpy="0.0 0.0 0.0" />
+        <origin xyz="0 0.450 -.03" rpy="0.0 0.0 0.0" />
       <parent link="${prefix}link_6" />
       <child link="${prefix}tool0" />
     </joint>
-        <!-- ROS-Industrial 'tool0' frame: all-zeros tool frame -->
-    <link name="${prefix}ee_link" />
-    <joint name="${prefix}ee_joint" type="fixed">
-      <!-- <origin xyz="0 0.020 0.0" rpy="0.0 ${-pi/2.0} ${-pi/2.0}" /> -->
-        <origin xyz="0 0.480 0.0" rpy="0.0 0.0 0.0" />
-      <parent link="${prefix}link_6" />
-      <child link="${prefix}ee_link" />
-    </joint>
   </xacro:macro>
 </robot>

File: hiwin_roller_support/urdf/roller_macro.xacro (robot description, xacro)
@@ -7,5 +7,5 @@
             <origin xyz="0 0 0" rpy="${pi/2} 0 ${pi}"/>
             <geometry>
-                <mesh filename="package://hiwin_roller_support/meshes/roller_mount.stl"  />
+                <mesh filename="package://hiwin_roller_support/meshes/hiwin_ee_base.stl"  scale="0.001 0.001 0.001"/>
             </geometry>
             <material name="LightGrey">
@@ -16,5 +16,22 @@
             <origin xyz="0 0 0" rpy="${pi/2} 0 ${pi}"/>
             <geometry>
-                <mesh filename="package://hiwin_roller_support/meshes/roller_mount.stl" />
+                <mesh filename="package://hiwin_roller_support/meshes/hiwin_ee_base.stl" scale="0.001 0.001 0.001"/>
+            </geometry>
+        </collision>
+    </link>
+    <link name="${prefix}link_0">
+        <visual>
+            <origin xyz="0.0 0.0 0.0" rpy="${pi/2} ${pi} 0"/>
+            <geometry>
+                <mesh filename="package://hiwin_roller_support/meshes/hiwin_ee_mount.stl" scale="0.001 0.001 0.001"/>
+            </geometry>
+            <material name="LightGrey">
+                <color rgba="0.7 0.7 0.7 1.0"/>
+            </material>
+        </visual>
+        <collision>
+            <origin xyz="0.0 0.0 0.0" rpy="${pi/2} ${pi} 0"/>
+            <geometry>
+                <mesh filename="package://hiwin_roller_support/meshes/hiwin_ee_mount.stl" scale="0.001 0.001 0.001"/>
             </geometry>
         </collision>
@@ -31,5 +48,5 @@
         </visual>
         <collision>
-            <origin xyz="0.0 0.0 0.0" rpy="${pi/2} 0 0"/>
+            <origin xyz="0.0 0.0 0.0" rpy="${pi/2} ${pi} 0"/>
             <geometry>
                 <mesh filename="package://hiwin_roller_support/meshes/roller.stl" scale="0.001 0.001 0.001"/>
@@ -43,6 +60,11 @@
     <!-- joints: main serial chain -->
     <joint name="${prefix}joint_1" type="fixed">
-        <origin xyz="0.0 0. 0.0" rpy="${pi} 0.0 0.0" />
+        <origin xyz="0.0 0.005 0.0" rpy="${pi} 0.0 0.0" />
         <parent link="${prefix}base_link" />
+        <child link="${prefix}link_0" />
+    </joint>
+    <joint name="${prefix}joint_2" type="fixed">
+        <origin xyz="0.0 0 0.0" rpy="0.0 0.0 0.0" />
+        <parent link="${prefix}link_0" />
         <child link="${prefix}link_1" />
     </joint>

Commit message: pedestal added

File: hiwin_ra610_1869_gb_support/urdf/ra610_1869_gb_macro.xacro (robot description, xacro)
@@ -3,5 +3,22 @@
 <xacro:macro name="manipulator" params="prefix">
     <!-- links: main serial chain -->
-    <link name="${prefix}base_link" >
+    <link name ="${prefix}base_link">
+        <visual>
+            <oriign xyz="0.1651 0.1651 0" rpy="0 0 {-pi/2}"/>
+            <geometry>
+                <mesh filename="package://hiwin_ra610_1869_gb_support/meshes/pedestal.stl" scale="0.001 0.001 0.001"/>
+            </geometry>
+            <material name="LightGrey">
+                <color rgba="0.999 0.999 0.999 1.0"/>
+            </material>
+        </visual>
+        <collision>
+            <oriign xyz="0 0 0" rpy="{pi/2} 0 0"/>
+            <geometry>
+                <mesh filename="package://hiwin_ra610_1869_gb_support/meshes/pedestal.stl" scale="0.001 0.001 0.001"/>
+            </geometry>
+        </collision>
+    </link>
+    <link name="${prefix}mount_link" >
         <visual>
             <origin xyz="0 0 0" rpy="0 0 ${pi/2}"/>
@@ -124,8 +141,13 @@
     <!-- end_effector frame -->
     <link name="${prefix}end_effector" />
+    <joint name="${prefix}joint_0" type="fixed">
+        <origin xyz="0 0 0.2413" rpy="0 0 0" />
+        <parent link="${prefix}base_link" />
+        <child link="${prefix}mount_link" />
+    </joint>
     <!-- joints: main serial chain -->
     <joint name="${prefix}joint_1" type="revolute">
         <origin xyz="0.0 0.0 0.1965" rpy="0.0 0.0 0.0" />
-        <parent link="${prefix}base_link" />
+        <parent link="${prefix}mount_link" />
         <child link="${prefix}link_1" />
         <axis xyz="0 0 1" />
@@ -189,6 +211,6 @@
     <link name="${prefix}tool0" />
     <joint name="${prefix}link_6-tool0" type="fixed">
-      <!-- <origin xyz="0 0.020 0.0" rpy="0.0 ${-pi/2.0} ${-pi/2.0}" /> -->
-        <origin xyz="0 0.450 -.03" rpy="0.0 0.0 0.0" />
+        <!-- <origin xyz="0 0.480 -.03" rpy="0.0 0.0 0.0" /> -->
+        <origin xyz="0 0.355 0" rpy="0.0 0.0 0.0" />
       <parent link="${prefix}link_6" />
       <child link="${prefix}tool0" />
