Commit message: smaller roller added

File: hiwin_ra610_1869_gb_support/urdf/ra610_1869_gb_macro.xacro (robot description, xacro)
@@ -3,22 +3,5 @@
 <xacro:macro name="manipulator" params="prefix">
     <!-- links: main serial chain -->
-    <link name ="${prefix}base_link">
-        <visual>
-            <oriign xyz="0.1651 0.1651 0" rpy="0 0 {-pi/2}"/>
-            <geometry>
-                <mesh filename="package://hiwin_ra610_1869_gb_support/meshes/pedestal.stl" scale="0.001 0.001 0.001"/>
-            </geometry>
-            <material name="LightGrey">
-                <color rgba="0.999 0.999 0.999 1.0"/>
-            </material>
-        </visual>
-        <collision>
-            <oriign xyz="0 0 0" rpy="{pi/2} 0 0"/>
-            <geometry>
-                <mesh filename="package://hiwin_ra610_1869_gb_support/meshes/pedestal.stl" scale="0.001 0.001 0.001"/>
-            </geometry>
-        </collision>
-    </link>
-    <link name="${prefix}mount_link" >
+    <link name="${prefix}base_link" >
         <visual>
             <origin xyz="0 0 0" rpy="0 0 ${pi/2}"/>
@@ -141,13 +124,8 @@
     <!-- end_effector frame -->
     <link name="${prefix}end_effector" />
-    <joint name="${prefix}joint_0" type="fixed">
-        <origin xyz="0 0 0.2413" rpy="0 0 0" />
-        <parent link="${prefix}base_link" />
-        <child link="${prefix}mount_link" />
-    </joint>
     <!-- joints: main serial chain -->
     <joint name="${prefix}joint_1" type="revolute">
         <origin xyz="0.0 0.0 0.1965" rpy="0.0 0.0 0.0" />
-        <parent link="${prefix}mount_link" />
+        <parent link="${prefix}base_link" />
         <child link="${prefix}link_1" />
         <axis xyz="0 0 1" />
@@ -190,5 +168,5 @@
     </joint>
     <joint name="${prefix}end_effector" type="fixed">
-        <origin xyz="0 0.450 0.0" rpy="0.0 0.0 0.0" />
+        <origin xyz="0 0.355 0.0" rpy="0.0 0.0 0.0" />
         <parent link="${prefix}link_6" />
         <child link="${prefix}end_effector" />

File: hiwin_roller_support/urdf/small_roller_macro.xacro (robot description, xacro)
@@ -17,21 +17,4 @@
             <geometry>
                 <mesh filename="package://hiwin_roller_support/meshes/hiwin_ee_base.stl" scale="0.001 0.001 0.001"/>
-            </geometry>
-        </collision>
-    </link>
-    <link name="${prefix}link_0">
-        <visual>
-            <origin xyz="0.0 0.0 0.0" rpy="${pi/2} ${pi} 0"/>
-            <geometry>
-                <mesh filename="package://hiwin_roller_support/meshes/pole.stl" scale="0.001 0.001 0.001"/>
-            </geometry>
-            <material name="LightGrey">
-                <color rgba="0.7 0.7 0.7 1.0"/>
-            </material>
-        </visual>
-        <collision>
-            <origin xyz="0.0 0.0 0.0" rpy="${pi/2} ${pi} 0"/>
-            <geometry>
-                <mesh filename="package://hiwin_roller_support/meshes/pole.stl" scale="0.001 0.001 0.001"/>
             </geometry>
         </collision>
@@ -62,9 +45,4 @@
         <origin xyz="0.0 0.005 0.0" rpy="${pi} 0.0 0.0" />
         <parent link="${prefix}base_link" />
-        <child link="${prefix}link_0" />
-    </joint>
-    <joint name="${prefix}joint_2" type="fixed">
-        <origin xyz="0.0 -0.005 0.0" rpy="0.0 0.0 0.0" />
-        <parent link="${prefix}link_0" />
         <child link="${prefix}link_1" />
     </joint>

File: hiwin_small_roller_support/urdf/small_roller_macro.xacro (robot description, xacro)
@@ -17,21 +17,4 @@
             <geometry>
                 <mesh filename="package://hiwin_roller_support/meshes/hiwin_ee_base.stl" scale="0.001 0.001 0.001"/>
-            </geometry>
-        </collision>
-    </link>
-    <link name="${prefix}link_0">
-        <visual>
-            <origin xyz="0.0 0.0 0.0" rpy="${pi/2} ${pi} 0"/>
-            <geometry>
-                <mesh filename="package://hiwin_roller_support/meshes/pole.stl" scale="0.001 0.001 0.001"/>
-            </geometry>
-            <material name="LightGrey">
-                <color rgba="0.7 0.7 0.7 1.0"/>
-            </material>
-        </visual>
-        <collision>
-            <origin xyz="0.0 0.0 0.0" rpy="${pi/2} ${pi} 0"/>
-            <geometry>
-                <mesh filename="package://hiwin_roller_support/meshes/pole.stl" scale="0.001 0.001 0.001"/>
             </geometry>
         </collision>
@@ -62,9 +45,4 @@
         <origin xyz="0.0 0.005 0.0" rpy="${pi} 0.0 0.0" />
         <parent link="${prefix}base_link" />
-        <child link="${prefix}link_0" />
-    </joint>
-    <joint name="${prefix}joint_2" type="fixed">
-        <origin xyz="0.0 -0.01 0.0" rpy="0.0 0.0 0.0" />
-        <parent link="${prefix}link_0" />
         <child link="${prefix}link_1" />
     </joint>
